File: PCB/Camera/Camera.kicad_pcb (KiCad board)
At the start: 2 copper layers, 85.5 x 66 mm, 3 parts, among them U4 ESP32-WROVER-E

Commit message: PCB changes
Parts:
- removed REF**: Camera_Interface, Camera_Components:Camera_Interface
- added C1: 0.1 uF, Capacitor_SMD:C_1206_3216Metric_Pad1.33x1.80mm_HandSolder, B.Cu at (176.5, 57.1)
- added C2: 15 pF, Capacitor_SMD:C_1206_3216Metric_Pad1.33x1.80mm_HandSolder, B.Cu at (194.9, 73.7)
- added C3: 0.1 uF, Capacitor_SMD:C_1206_3216Metric_Pad1.33x1.80mm_HandSolder, B.Cu at (187.3, 73.7)
- added C4: 0.1 uF, Capacitor_SMD:C_1206_3216Metric_Pad1.33x1.80mm_HandSolder, B.Cu at (192.4, 73.7)
- added C5: 10 uF, Capacitor_SMD:C_1206_3216Metric_Pad1.33x1.80mm_HandSolder, B.Cu at (176.5, 47.6)
- added C6: 22 uF, Capacitor_SMD:C_1206_3216Metric_Pad1.33x1.80mm_HandSolder, F.Cu at (202.6, 68.6)
- added C7: 22 uF, Capacitor_SMD:C_1206_3216Metric_Pad1.33x1.80mm_HandSolder, F.Cu at (172.1, 68.6)
- added C8: 0.1 uF, Capacitor_SMD:C_1206_3216Metric_Pad1.33x1.80mm_HandSolder, B.Cu at (176.5, 50.8)
- added R1: 10K, Resistor_SMD:R_1206_3216Metric_Pad1.30x1.75mm_HandSolder, B.Cu at (176.5, 54.0)
- added R2: 10K, Resistor_SMD:R_1206_3216Metric_Pad1.30x1.75mm_HandSolder, B.Cu at (176.5, 44.5)
- added R3: 1K, Resistor_SMD:R_1206_3216Metric_Pad1.30x1.75mm_HandSolder, B.Cu at (189.9, 73.7)
- added R4: 4.7K, Resistor_SMD:R_1206_3216Metric_Pad1.30x1.75mm_HandSolder, B.Cu at (184.8, 73.7)
- added R5: 4.7K, Resistor_SMD:R_1206_3216Metric_Pad1.30x1.75mm_HandSolder, B.Cu at (179.7, 73.7)
- added R6: 4.7K, Resistor_SMD:R_1206_3216Metric_Pad1.30x1.75mm_HandSolder, B.Cu at (182.2, 73.7)
- added SW1: SW_Push, Camera_Components:6x6x4.3 SMD button, F.Cu at (199.4, 55.2)
- added SW2: SW_Push, Camera_Components:6x6x4.3 SMD button, F.Cu at (199.4, 46.4)
- added U2: ~, PCM_Espressif:ESP32-WROVER-E, B.Cu at (196.8, 50.8)
- added U3: ~, Camera_Components:24-pin-FPC-0.5mm, F.Cu at (187.3, 73.7)
- added U5: ~, PCM_Espressif:ESP32-WROVER-E, F.Cu at (177.8, 50.8)
- added U6: AMS1117-2.85, Package_TO_SOT_SMD:SOT-223-3_TabPin2, F.Cu at (174.0, 73.7)
- U4: value ESP32-WROVER-E -> AMS1117-1.2; footprint PCM_Espressif:ESP32-WROVER-E -> Package_TO_SOT_SMD:SOT-223-3_TabPin2
- moved U4 44.2 mm to (200.7, 73.7), turned to 180 degrees
- moved U1 6.51 mm to (187.3, 38.5), turned to 90 degrees
Connections:
- U1 pad 1: GNDREF -> /B_TX
- U1 pad 2: /FLASH TX -> /B_RX
- U1 pad 3: /FLASH RX -> unconnected-(U1-5V-Pad3)
- U1 pad 4: /3.3V -> GNDREF
- U1 pad 5: unconnected-(U1-5V-Pad5) -> /3.3V
- U4 pad 2: /3.3V -> /1.2V
- U4 pad 3: /EN -> /3.3V
Routing:
- net GNDREF: track 6.50 -> 236.6 mm, vias 0 -> 13
- net /3.3V: track 0.00 -> 131.3 mm, vias 0 -> 8
- net /B_EN: track 0.00 -> 52.7 mm, vias 0 -> 4
- net /CAM_DATA3: track 0.00 -> 37.3 mm
- net /CAM_DATA4: track 0.00 -> 37.0 mm
- net /B_IO0: track 0.00 -> 33.3 mm, vias 0 -> 2
- net /1.2V: track 0.00 -> 27.4 mm
- net /CAM_PCLK: track 0.00 -> 26.2 mm, vias 0 -> 1
- net /2.8V: track 0.00 -> 25.9 mm, vias 0 -> 2
- net /CAM_SIOD: track 0.00 -> 25.5 mm, vias 0 -> 1
- net /CAM_SIOC: track 0.00 -> 21.6 mm
- net /CAM_VSYNC: track 0.00 -> 21.5 mm
- net /CAM_HREF: track 0.00 -> 21.4 mm
- net /CAM_DATA9: track 0.00 -> 20.6 mm
- net /CAM_XCLK: track 0.00 -> 19.7 mm
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Other:
- board outline removed

Commit message: PCB changes
Parts:
- removed C6, C7: 22 uF, Capacitor_SMD:C_1206_3216Metric_Pad1.33x1.80mm_HandSolder
- removed U4: AMS1117-1.2, Package_TO_SOT_SMD:SOT-223-3_TabPin2
- removed U6: AMS1117-2.85, Package_TO_SOT_SMD:SOT-223-3_TabPin2
- added C10: 1 uF, Capacitor_SMD:C_1206_3216Metric_Pad1.33x1.80mm_HandSolder, F.Cu at (200.0, 66.7)
- added C11: 1 uF, Capacitor_SMD:C_1206_3216Metric_Pad1.33x1.80mm_HandSolder, F.Cu at (174.6, 66.7)
- added D1: LED, Camera_Components:vibration motor, F.Cu at (215.5, 78.0)
- added Q1: S8050, Camera_Components:transistor, B.Cu at (192.4, 64.1)
- added Q2: S8050, Camera_Components:transistor, F.Cu at (211.1, 79.5)
- added R7: 4.7K, Resistor_SMD:R_1206_3216Metric_Pad1.30x1.75mm_HandSolder, B.Cu at (193.0, 67.9)
- added R8: 4.7K, Resistor_SMD:R_1206_3216Metric_Pad1.30x1.75mm_HandSolder, F.Cu at (206.0, 79.0)
- added U10: ~, Camera_Components:XC6206, F.Cu at (177.8, 69.2)
- added U7: ~, Camera_Components:vibration motor, B.Cu at (187.3, 66.0)
- added U8: ~, Camera_Components:XC6206, F.Cu at (196.8, 69.2)
- renumbered SW2 to BOOT1, U3 to CAMERA1, SW1 to RESET1
Connections:
- U2 pad 13: unconnected-(U2-IO14-Pad13) -> /V_CTRL
- U2 pad 8: unconnected-(U2-IO32-Pad8) -> /LED_CTRL
Routing:
- net /V_CTRL: track 0.00 -> 11.5 mm
- net /2.8V: track 25.9 -> 16.5 mm, vias 2 -> 0
- net GNDREF: track 236.6 -> 228.5 mm
- net /3.3V: track 131.3 -> 124.1 mm, vias 8 -> 9
- net /1.2V: track 27.4 -> 21.6 mm
- net /CAM_SIOD: track 25.5 -> 24.5 mm
- net /CAM_VSYNC: track 21.5 -> 20.6 mm
- net /CAM_HREF: track 21.4 -> 20.5 mm
- net /CAM_SIOC: track 21.6 -> 20.7 mm
- net /CAM_DATA9: track 20.6 -> 20.0 mm
Other:
- board outline added: 39.4 x 41.9 mm

Commit message: Added a BUTTON hell yeah
Parts:
- added GEN1: SW_Push, Camera_Components:6x6x4.3 SMD button, B.Cu at (174.0, 64.8)
- added R9: 10K, Resistor_SMD:R_1206_3216Metric_Pad1.30x1.75mm_HandSolder, B.Cu at (181.0, 64.8)
- R8: moved to B.Cu
- moved Q2 21.4 mm to (196.8, 63.5), turned to 90 degrees
- moved D1 17.6 mm to (203.2, 65.4), turned to -90 degrees
- moved R8 12.3 mm to (200.7, 67.9), turned to 180 degrees
- moved U1 0.87 mm to (187.3, 39.4)
Connections:
- U2 pad 11: unconnected-(U2-IO26-Pad11) -> /V_CTRL
- U2 pad 12: unconnected-(U2-IO27-Pad12) -> /GEN_BTN
- U2 pad 13: /V_CTRL -> unconnected-(U2-IO14-Pad13)
Routing:
- net /GEN_BTN: track 0.00 -> 24.6 mm
- net /3.3V: track 124.1 -> 129.6 mm
- net Net-(D1-A): track 0.00 -> 4.76 mm, vias 0 -> 1
- net Net-(Q1-E): track 0.00 -> 4.58 mm
- net Net-(Q2-E): track 0.00 -> 4.38 mm, vias 0 -> 1
- net GNDREF: track 228.5 -> 232.3 mm, vias 13 -> 12
- net /LED_CTRL: track 0.00 -> 3.15 mm, vias 0 -> 1
- net /V_CTRL: track 11.5 -> 9.30 mm
- net /CAM_SIOC: track 20.7 -> 22.0 mm, vias 0 -> 1
- net /CAM_PCLK: track 26.2 -> 25.3 mm
- net /CAM_PWDN: track 7.00 -> 6.43 mm
- net /CAM_DATA5: track 17.5 -> 16.9 mm
- net /B_RX: track 9.40 -> 8.87 mm
Other:
- board text added: "3.3V"
- board text added: "B_RX"
- board text added: "B_TX"
- board text added: "GND"
- board text added: "NC"
- board text added: "W_RX"
- board text added: "W_TX"

Commit message: Finalized PCB design
Other:
- board text added: "3V3"
- board text added: "BRX"
- board text added: "BTX"
- board text added: "WRX"
- board text added: "WTX"
- board text removed: "3.3V"
- board text removed: "B_RX"
- board text removed: "B_TX"
- board text removed: "W_RX"
- board text removed: "W_TX"
Changed lines of the file:
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@@
 	)
 	(setup
+		(stackup
+			(layer "F.SilkS"
+				(type "Top Silk Screen")
+			)
+			(layer "F.Paste"
+				(type "Top Solder Paste")
+			)
+			(layer "F.Mask"
+				(type "Top Solder Mask")
+				(color "Blue")
+				(thickness 0.01)
+			)
+			(layer "F.Cu"
+				(type "copper")
+				(thickness 0.035)
+			)
+			(layer "dielectric 1"
+				(type "core")
+				(thickness 1.51)
+				(material "FR4")
+				(epsilon_r 4.5)
+				(loss_tangent 0.02)
+			)
+			(layer "B.Cu"
+				(type "copper")
+				(thickness 0.035)
+			)
+			(layer "B.Mask"
+				(type "Bottom Solder Mask")
+				(color "Blue")
+				(thickness 0.01)
+			)
+			(layer "B.Paste"
+				(type "Bottom Solder Paste")
+			)
+			(layer "B.SilkS"
+				(type "Bottom Silk Screen")
+			)
+			(copper_finish "None")
+			(dielectric_constraints no)
+		)
 		(pad_to_mask_clearance 0)
 		(allow_soldermask_bridges_in_footprints no)
@@
 			(plotinvisibletext no)
 			(sketchpadsonfab no)
-			(subtractmaskfromsilk no)
+			(subtractmaskfromsilk yes)
 			(outputformat 1)
 			(mirror no)
-			(drillshape 1)
+			(drillshape 0)
 			(scaleselection 1)
-			(outputdirectory "")
+			(outputdirectory "C:/SD/visionbuzz/PCB/Camera/gerber/")
 		)
 	)
@@
 		(layer "Edge.Cuts")
 	)
-	(gr_text "W_RX"
-		(at 182.245 37.846 180)
+	(gr_text "WRX"
+		(at 180.975 37.846 180)
 		(layer "F.SilkS")
 		(effects
 			(font
-				(size 0.508 0.508)
-				(thickness 0.0762)
+				(size 0.8128 0.8128)
+				(thickness 0.08128)
 			)
 		)
@@
 		(effects
 			(font
-				(size 0.508 0.508)
-				(thickness 0.0762)
+				(size 0.8128 0.8128)
+				(thickness 0.08128)
 			)
 		)
 	)
-	(gr_text "B_RX"
-		(at 192.405 37.846 180)
+	(gr_text "BRX"
+		(at 193.675 37.846 180)
 		(layer "F.SilkS")
 		(effects
 			(font
-				(size 0.508 0.508)
-				(thickness 0.0762)
+				(size 0.8128 0.8128)
+				(thickness 0.08128)
 			)
 		)
 	)
-	(gr_text "W_TX"
-		(at 179.705 37.846 180)
+	(gr_text "WTX"
+		(at 177.165 39.37 180)
 		(layer "F.SilkS")
 		(effects
 			(font
-				(size 0.508 0.508)
-				(thickness 0.0762)
+				(size 0.8128 0.8128)
+				(thickness 0.08128)
 			)
 		)
 	)
-	(gr_text "3.3V"
-		(at 184.785 37.846 180)
+	(gr_text "3V3"
+		(at 184.15 37.846 180)
 		(layer "F.SilkS")
 		(effects
 			(font
-				(size 0.508 0.508)
-				(thickness 0.0762)
+				(size 0.8128 0.8128)
+				(thickness 0.08128)
 			)
 		)
 	)
-	(gr_text "B_TX"
-		(at 194.945 37.846 180)
+	(gr_text "BTX"
+		(at 197.485 39.37 180)
 		(layer "F.SilkS")
 		(effects
 			(font
-				(size 0.508 0.508)
-				(thickness 0.0762)
+				(size 0.8128 0.8128)
+				(thickness 0.08128)
 			)
 		)
 	)
 	(gr_text "NC"
-		(at 189.865 37.846 180)
+		(at 190.5 37.846 180)
 		(layer "F.SilkS")
 		(effects
 			(font
-				(size 0.508 0.508)
-				(thickness 0.0762)
+				(size 0.8128 0.8128)
+				(thickness 0.08128)
 			)
 		)
@@
 	(segment
 		(start 200.5 40.5)
-		(end 201.295 41.295)
+		(end 196.075 40.5)
 		(width 0.2)
 		(layer "B.Cu")
@@
 	)
 	(segment
-		(start 201.295 41.295)
-		(end 201.295 42.05)
+		(start 196.075 40.5)
+		(end 194.945 39.37)
 		(width 0.2)
 		(layer "B.Cu")
@@
 	)
 	(segment
-		(start 196.945 40.5)
-		(end 200.5 40.5)
+		(start 201.295 42.05)
+		(end 201.295 41.295)
 		(width 0.2)
 		(layer "B.Cu")
@@
 	)
 	(segment
-		(start 194.945 38.5)
-		(end 196.945 40.5)
+		(start 201.295 41.295)
+		(end 200.5 40.5)
 		(width 0.2)
 		(layer "B.Cu")
@@
 	)
 	(segment
-		(start 192.405 38.5)
-		(end 194.905 41)
+		(start 200.025 41.525)
+		(end 199.5 41)
 		(width 0.2)
 		(layer "B.Cu")
@@
 	)
 	(segment
-		(start 199.5 41)
-		(end 200.025 41.525)
+		(start 194.035 41)
+		(end 192.405 39.37)
 		(width 0.2)
 		(layer "B.Cu")
@@
 	)
 	(segment
-		(start 194.905 41)
-		(end 199.5 41)
+		(start 199.5 41)
+		(end 194.035 41)
 		(width 0.2)
 		(layer "B.Cu")

Commit message: integration stuff
Parts:
- moved GEN1 0.64 mm to (174.0, 65.4)
Connections:
- U5 pad 10: /CAM_DATA8 -> /CAM_VSYNC
- U5 pad 11: /CAM_DATA7 -> /CAM_HREF
- U5 pad 12: /CAM_PCLK -> /CAM_XCLK
- U5 pad 13: /CAM_DATA6 -> /CAM_PCLK
- U5 pad 4: /CAM_SIOD -> /CAM_DATA9
- U5 pad 5: /CAM_SIOC -> /CAM_DATA8
- U5 pad 6: /CAM_VSYNC -> /CAM_DATA7
- U5 pad 7: /CAM_HREF -> /CAM_DATA6
- U5 pad 8: /CAM_DATA9 -> /CAM_SIOD
- U5 pad 9: /CAM_XCLK -> /CAM_SIOC
Routing:
- net /CAM_DATA7: track 19.3 -> 29.1 mm, vias 0 -> 4
- net /CAM_DATA6: track 18.6 -> 28.0 mm, vias 0 -> 4
- net /CAM_DATA8: track 19.4 -> 27.7 mm, vias 0 -> 2
- net /CAM_DATA9: track 19.6 -> 24.4 mm, vias 0 -> 2
- net GNDREF: track 232.3 -> 229.1 mm
- net /CAM_SIOD: track 24.4 -> 21.4 mm
- net /CAM_HREF: track 20.5 -> 17.8 mm
- net /CAM_VSYNC: track 20.6 -> 17.9 mm
- net /CAM_SIOC: track 22.0 -> 19.9 mm
- net /CAM_DATA2: track 18.3 -> 19.5 mm
- net /CAM_XCLK: track 19.7 -> 18.5 mm
- net /GEN_BTN: track 24.6 -> 24.0 mm
